File: jetson_imu_board/jetson_imu_board.kicad_pcb (KiCad board)
At the start: 2 copper layers, 12 parts, among them P1 J3A1, P2 J3A2, P3 CONN_01X02, P4 CONN_01X04, P5 CONN_01X06, P6 CONN_01X07, U1 TXB0108

Commit message: Finished routing and layout
Parts:
- removed P1: J3A1, Pin_Headers:Pin_Header_Straight_2x25_Pitch2.00mm
- removed P2: J3A2, Pin_Headers:Pin_Header_Straight_2x25_Pitch2.00mm
- removed P3: CONN_01X02, Pin_Headers:Pin_Header_Straight_1x02
- added Address: CONN_01X02, Pin_Headers:Pin_Header_Straight_1x02, F.Cu at (87.6, 52.6)
- added JA31: J3A1, Pin_Headers:Pin_Header_Straight_2x25_Pitch2.00mm, B.Cu at (88.0, 67.0)
- added JA32: J3A2, jetson_imu_footprints:Pin_Header_Straight_3x25_Pitch2.00mm, B.Cu at (88.0, 63.0)
- moved C1 173.2 mm to (48.8, 45.9), turned to 270 degrees
- moved C2 163.5 mm to (48.8, 53.2), turned to 270 degrees
- moved U1 162.8 mm to (54.5, 49.0)
- moved C3 160.0 mm to (54.8, 43.8), turned to 180 degrees
- moved R1 159.0 mm to (54.0, 55.5)
- moved P4 141.1 mm to (68.6, 53.3), turned to 90 degrees
- moved R2 132.4 mm to (88.0, 47.0), turned to 90 degrees
- moved P6 130.6 mm to (67.6, 44.5), turned to 90 degrees
- moved P5 126.0 mm to (66.0, 71.1), turned to 90 degrees
Connections:
- net +3V3 renamed /JET_3V3
- net /IMU_3VO renamed Net-(P5-Pad2)
- net /IMU_INT renamed Net-(P4-Pad3)
- net /IMU_PS0 renamed Net-(P4-Pad1)
- net /IMU_PS1 renamed Net-(P4-Pad2)
- net GND renamed /JET_GND
- P5 pad 4: /IMU_SDA -> /JET_SDA
- P5 pad 5: /IMU_SCL -> /JET_SCL
Routing:
- net /JET_3V3: track 0.00 -> 96.4 mm, vias 0 -> 2
- net /JET_1V8: track 0.00 -> 59.6 mm, vias 0 -> 2
- net /IMU_RST: track 0.00 -> 46.3 mm
- net /JET_AMS_1V8: track 0.00 -> 36.4 mm, vias 0 -> 4
- net /JET_GND: track 0.00 -> 30.0 mm, vias 0 -> 6
- net /GPIO166_3V3: track 0.00 -> 28.9 mm
- net /JET_GPIO57: track 0.00 -> 28.6 mm
- net /GPIO165_3V3: track 0.00 -> 26.1 mm
- net /JET_GPIO162: track 0.00 -> 24.9 mm
- net /JET_GPIO161: track 0.00 -> 24.1 mm
- net /JET_GPIO160: track 0.00 -> 23.8 mm
- net /GPIO164_3V3: track 0.00 -> 23.3 mm
- net /IMU_ADR: track 0.00 -> 22.2 mm
- net /GPIO163_3V3: track 0.00 -> 20.6 mm
- net /GPIO162_3V3: track 0.00 -> 17.9 mm
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- added copper zone on B.Cu, net /JET_GND
Other:
- board outline added: 53.4 x 32 mm
- net class Default: clearance 0.2 -> 0.1524; trace_width 0.25 -> 0.1524; via_dia 0.6 -> 0.6858; via_drill 0.4 -> 0.3302
- net class Signal added: clearance 0.1524, trace_width 0.254, via_dia 0.6858, via_drill 0.3302
- rule trace_clearance: 0.2 -> 0.1524
- rule trace_min: 0.2 -> 0.1524
- rule via_min_drill: 0.3 -> 0.3302
- rule via_min_size: 0.4 -> 0.6858
